File: cad/pcb/cpu/v1.0/jimduino.sch (EAGLE design)
At the start: 62 parts, among them CN1 SM02B-SRSS-TB, P1 DF12-32-DP, P2 DF12-32-DP, Q1 FDN360P, Q2 FDN360P, SW1 SWITCH-MOMENTARY-2SMD-REDUNDA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, U1 STM32F415R, U2 MCP1703, U3 MCP73831, U4 LTC2954-2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

Commit message: unknown changes
Parts:
- C12, C13: value 4pF -> 8pF
- U$1: value USB-CON-5PIN-105017-0001 -> MICROUSB; device GeekAmmo:USB-CON-5PIN-105017-0001 -> jimduino:MICROUSB
Connections:
- net GND: now also U$1.SH1, U$1.SH2, U$1.SH3, U$1.SH4, U$1.SH5, U$1.SH6
Changed lines of the file:
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@@
 <part name="U2" library="linear" deviceset="MCP1703" device=""/>
 <part name="C11" library="SparkFun-Capacitors" deviceset="CAP" device="0805" value="1uF"/>
-<part name="C12" library="SparkFun-Capacitors" deviceset="CAP" device="0402-CAP" value="4pF"/>
-<part name="C13" library="SparkFun-Capacitors" deviceset="CAP" device="0402-CAP" value="4pF"/>
+<part name="C12" library="SparkFun-Capacitors" deviceset="CAP" device="0402-CAP" value="8pF"/>
+<part name="C13" library="SparkFun-Capacitors" deviceset="CAP" device="0402-CAP" value="8pF"/>
 <part name="Y2" library="SparkFun-FreqCtrl" deviceset="CRYSTAL" device="EPSONMC146" value="32.768kHz (9pF)"/>
 <part name="C14" library="SparkFun-Capacitors" deviceset="CAP" device="0805" value="1uF"/>
@@
 <part name="R14" library="SparkFun-Passives" deviceset="RESISTOR" device="0805-RES" value="0k"/>
 <part name="C22" library="SparkFun-Capacitors" deviceset="CAP" device="0805" value="0.1uF"/>
-<part name="U$1" library="GeekAmmo" deviceset="USB-CON-5PIN" device="-105017-0001"/>
+<part name="U$1" library="jimduino" deviceset="MICROUSB" device=""/>
 </parts>
 <sheets>
@@
 <attribute name="VALUE" x="-16.764" y="137.541" size="1.778" layer="96"/>
 </instance>
-<instance part="U$1" gate="G$1" x="111.76" y="48.26" rot="MR0"/>
+<instance part="U$1" gate="G$1" x="114.3" y="48.26"/>
 </instances>
 <busses>
@@
 <segment>
 <wire x1="-7.62" y1="91.44" x2="-15.24" y2="91.44" width="0.1524" layer="91"/>
-<label x="-14.478" y="92.202" size="1.778" layer="95"/>
+<label x="-16.51" y="91.948" size="1.778" layer="95"/>
 <pinref part="R14" gate="G$1" pin="1"/>
 </segment>
@@
 </segment>
 <segment>
+<pinref part="U$1" gate="G$1" pin="SH1"/>
+<pinref part="U$1" gate="G$1" pin="SH6"/>
 <wire x1="127" y1="53.34" x2="127" y2="50.8" width="0.1524" layer="91"/>
 <label x="129.54" y="50.8" size="1.778" layer="95"/>
+<pinref part="U$1" gate="G$1" pin="SH2"/>
+<junction x="127" y="50.8"/>
 <wire x1="127" y1="50.8" x2="127" y2="48.26" width="0.1524" layer="91"/>
+<pinref part="U$1" gate="G$1" pin="SH3"/>
+<junction x="127" y="48.26"/>
 <wire x1="127" y1="48.26" x2="127" y2="45.72" width="0.1524" layer="91"/>
+<pinref part="U$1" gate="G$1" pin="SH4"/>
+<junction x="127" y="45.72"/>
 <wire x1="127" y1="45.72" x2="127" y2="43.18" width="0.1524" layer="91"/>
+<pinref part="U$1" gate="G$1" pin="SH5"/>
+<junction x="127" y="43.18"/>
 <wire x1="127" y1="43.18" x2="127" y2="40.64" width="0.1524" layer="91"/>
 </segment>
