File: cad/pcb/eagle/breakout/breakout.brd (EAGLE design)
At the start: 38 x 31 mm, 9 parts, among them J1 DF12-32-DS, J2 DF12-32-DS

Commit message: Tweak board
Routing:
- net PC0: track 0.00 -> 38.8 mm, vias 0 -> 3
- net PA9: track 0.00 -> 37.6 mm, vias 0 -> 3
- net VCC: track 95.3 -> 58.5 mm, vias 4 -> 7
- net PA3: track 28.1 -> 55.9 mm, vias 1 -> 2
- net PA13: track 26.9 -> 47.7 mm, vias 2 -> 3
- net PA7: track 31.4 -> 50.1 mm
- net PC5: track 51.1 -> 68.2 mm, vias 5 -> 2
- net PB3: track 16.5 -> 32.9 mm, vias 1 -> 2
- net PC10: track 43.9 -> 57.8 mm, vias 2 -> 3
- net RESET#: track 62.2 -> 49.3 mm, vias 5 -> 6
- net PB12: track 55.0 -> 42.3 mm, vias 3 -> 2
- net PC4: track 50.2 -> 62.5 mm, vias 1 -> 9
- net PC9: track 18.8 -> 30.7 mm, vias 1 -> 4
- net PC3: track 24.1 -> 35.9 mm, vias 1 -> 2
- net PD2: track 27.1 -> 37.8 mm, vias 2 -> 3
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
Commit message: More board tweaks
Routing:
- net PWR_ON: track 72.8 -> 0.00 mm, vias 4 -> 0
- net VCC_3V3: track 72.2 -> 0.00 mm, vias 4 -> 0
- net PB14: track 60.1 -> 0.00 mm, vias 4 -> 0
- net VCC: track 58.5 -> 0.00 mm, vias 7 -> 0
- net PA7: track 50.1 -> 0.00 mm, vias 3 -> 0
- net RESET#: track 49.3 -> 0.00 mm, vias 6 -> 0
- net PA13: track 47.7 -> 0.00 mm, vias 3 -> 0
- net PB12: track 42.3 -> 0.00 mm, vias 2 -> 0
- net PB15: track 40.0 -> 0.00 mm, vias 6 -> 0
- net PD2: track 37.8 -> 0.00 mm, vias 3 -> 0
- net PA9: track 37.6 -> 73.3 mm, vias 3 -> 1
- net PB13: track 33.9 -> 0.00 mm
- net PC10: track 57.8 -> 24.1 mm, vias 3 -> 1
- net PB3: track 32.9 -> 0.00 mm, vias 2 -> 0
- net RSV0: track 32.8 -> 0.07 mm, vias 1 -> 0
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
Commit message: Better routing
Connections:
- net GND: now also PA8_15.3, PA8_15.4, PA8_15.5, PWR.6; no longer PWR.8
- net VCC: now also PWR.8; no longer PWR.4, PWR.5
- net VCC_3V3: now also PWR.4, PWR.5
Routing:
- net PB15: track 0.00 -> 57.9 mm, vias 0 -> 2
- net PWR_ON: track 0.00 -> 53.3 mm, vias 0 -> 6
- net VCC: track 0.00 -> 48.1 mm, vias 0 -> 2
- net PB14: track 0.00 -> 44.0 mm, vias 0 -> 3
- net PB12: track 0.00 -> 40.0 mm, vias 0 -> 1
- net RSV0: track 0.07 -> 36.5 mm, vias 0 -> 3
- net VCC_3V3: track 0.00 -> 36.4 mm, vias 0 -> 4
- net PA7: track 0.00 -> 34.7 mm, vias 0 -> 1
- net PB13: track 0.00 -> 33.8 mm, vias 0 -> 2
- net RESET#: track 0.00 -> 33.7 mm, vias 0 -> 4
- net PA6: track 0.00 -> 32.5 mm, vias 0 -> 1
- net RSV1: track 30.6 -> 61.3 mm, vias 1 -> 2
- net PA5: track 0.00 -> 30.5 mm, vias 0 -> 4
- net PA9: track 73.3 -> 42.9 mm, vias 1 -> 2
- net PC7: track 0.00 -> 28.3 mm, vias 0 -> 4
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Other:
- board text added: "A0"
- board text added: "A1"
- board text added: "A13"
- board text added: "A14"
- board text added: "A15"
- board text added: "A2"
- board text added: "A3"
- board text added: "A4"
- board text added: "A5"
- board text added: "A6"
- board text added: "A7"
- board text added: "A8"
- board text added: "A9"
- board text added: "B0"
- board text added: "B1"
- board text added: "B10"
- board text added: "B11"
- board text added: "B12"
- board text added: "B13"
- board text added: "B14"
- board text added: "B15"
- board text added: "B2"
- board text added: "B3"
- board text added: "B4"
- board text added: "B5"
- board text added: "B6"
- board text added: "B7"
- board text added: "B8"
- board text added: "B9"
- board text added: "C0"
- board text added: "C1"
- board text added: "C10"
- board text added: "C11"
- board text added: "C12"
- board text added: "C13"
- board text added: "C2"
- board text added: "C3"
- board text added: "C4"
- board text added: "C5"
- board text added: "C6"
- board text added: "C7"
- board text added: "C8"
- board text added: "C9"
- board text added: "GND"
- board text added: "MatchBox Breakout"
- board text added: "PD2"
- board text added: "PWR"
- board text added: "RS0"
- board text added: "RS1"
- board text added: "RST"
- board text added: "VCC"
- board text added: "VCC3"
- board text removed: "IO Breakout Board"
