File: cad/pcb/eagle/breakout/matchbox_bob_v10.brd (EAGLE design)
At the start: 40 x 32 mm, 9 parts, among them J1 DF12-32-DS, J2 DF12-32-DS

Commit message: Tweaks to BOB v1.0
Parts:
- added P1, P2: DF12-32-DP, micro1292:DF12-32-DP
Connections:
- new net RSV2: J2.17, P2.17
- new net RSV3: J2.19, P2.19
- net GND: now also P1.2, P1.4, P2.2, P2.4
- net PA0: now also P2.26
- net PA1: now also P2.24
- net PA13: now also P2.6
- net PA14: now also P1.11
- net PA15: now also P1.27
- net PA2: now also P2.22
- net PA3: now also P2.20
- net PA4: now also P2.27
- net PA5: now also P2.25
- net PA6: now also P2.23
- net PA7: now also P2.21
- net PA8: now also P2.8
- net PA9: now also P1.8
- net PB0: now also P2.15
- net PB1: now also P2.13
- net PB10: now also P2.9
- net PB11: now also P2.7
- net PB12: now also P2.18
- net PB13: now also P2.16
- net PB14: now also P2.14
- net PB15: now also P2.12
- net PB2: now also P2.11
- net PB3: now also P1.17
- net PB4: now also P1.15
- net PB5: now also P1.13
- net PB6: now also P1.9
- net PB7: now also P1.7
- net PB8: now also P1.5
- net PB9: now also P1.3
- net PC0: now also P1.12
- net PC1: now also P1.14
- net PC10: now also P1.25
- net PC11: now also P1.23
- net PC12: now also P1.21
- net PC13: now also P1.6
- net PC2: now also P1.16
- net PC3: now also P1.18
- net PC4: now also P1.20; no longer J2.19
- net PC5: now also P1.22; no longer J2.17
- net PC6: now also P1.24
- net PC7: now also P1.26
- net PC8: now also P1.10
- net PC9: now also P2.10
- net PD2: now also P1.19
- net PWR_ON: now also P1.28, P2.28
- net RESET#: now also P1.1, P2.1
- net RSV0: now also P2.3
- net RSV1: now also P2.5
- net VCC: now also P1.30, P1.32, P2.30, P2.32
- net VCC_3V3: now also P1.29, P1.31, P2.29, P2.31
Routing:
- net GND: track 0.00 -> 61.2 mm, vias 8 -> 11
- net RESET#: track 33.7 -> 71.6 mm, vias 4 -> 5
- net RSV1: track 61.3 -> 32.7 mm, vias 2 -> 3
- net PC10: track 28.5 -> 52.6 mm, vias 6 -> 3
- net VCC: track 48.1 -> 71.0 mm, vias 2 -> 6
- net PC5: track 62.7 -> 42.3 mm, vias 6 -> 3
- net PB12: track 40.0 -> 23.1 mm, vias 1 -> 2
- net PB15: track 57.9 -> 44.3 mm, vias 2 -> 5
- net PC11: track 24.2 -> 36.7 mm, vias 3 -> 2
- net PWR_ON: track 53.3 -> 63.9 mm, vias 6 -> 4
- net PB7: track 22.2 -> 11.8 mm, vias 2 -> 1
- net PA6: track 32.5 -> 42.7 mm, vias 1 -> 3
- net PB5: track 20.3 -> 13.5 mm, vias 2 -> 3
- net PA15: track 15.2 -> 8.36 mm, vias 2 -> 1
- net PB6: track 19.7 -> 13.2 mm
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Other:
- board text added: "MatchBox BOB V1.0"
- board text removed: "MatchBox Breakout"

Commit message: Add passthrough to v1.0 BOB
Connections:
- net PC4: now also J2.19
- net PC5: now also J2.17
- net RSV2: no longer J2.17
- net RSV3: no longer J2.19
Routing:
- net PA4: track 22.4 -> 64.0 mm, vias 3 -> 1
- net GND: track 61.2 -> 97.4 mm, vias 11 -> 0
- net RESET#: track 71.6 -> 36.1 mm, vias 5 -> 2
- net PB12: track 23.1 -> 48.1 mm, vias 2 -> 1
- net PC4: track 40.4 -> 61.1 mm, vias 2 -> 4
- net PWR_ON: track 63.9 -> 44.2 mm, vias 4 -> 2
- net PB14: track 47.3 -> 27.9 mm, vias 4 -> 1
- net PC10: track 52.6 -> 34.3 mm, vias 3 -> 1
- net PB5: track 13.5 -> 31.4 mm, vias 3 -> 1
- net PB4: track 15.7 -> 32.8 mm
- net PC5: track 42.3 -> 58.9 mm, vias 3 -> 4
- net PA9: track 47.0 -> 32.0 mm, vias 5 -> 2
- net PB15: track 44.3 -> 30.9 mm, vias 5 -> 1
- net PC11: track 36.7 -> 24.5 mm
- net PA8: track 14.3 -> 25.3 mm, vias 1 -> 0
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- added copper zone on layer 2, net GND
- added copper zone on layer 15, net VCC_3V3
Other:
- board text added: "MatchBox Breakout"
- board text removed: "MatchBox BOB V1.0"
